File: can-hat-r1.sch (KiCad schematic (older format))
At the start: 57 parts, among them P1 PINBALL-CONNECTOR, P2 PINBALL-CONNECTOR, P3 PIHAT, Q1 DMG2305UX, Q2 DMMT5401, U1 MCP2562, U2 MCP2515, U3 AP3513E, U4 CAT24C32, X1 CRYSTAL

Commit message: Updated to latest version of KiCAD. Added PDF of schematic.
Parts:
- C1, C14, C15, C16, C2, C3, C4, C5, C6, C7, C8, C9: symbol C -> C-RESCUE-can-hat-r1
- C10, C11, C12, C13: symbol CP -> CP-RESCUE-can-hat-r1
- D2, D3, D4: symbol LED -> LED-RESCUE-can-hat-r1
- R1, R10, R11, R12, R13, R14, R15, R16, R17, R18, R19, R2, R20, R21, R22, R23, R24, R3, R4, R5, R6, R7, R8, R9: symbol R -> R-RESCUE-can-hat-r1
Connections:
- net at U1.1 (CANTX): now also U2.1 (CANTX); no longer U2.2 (CANRX)
- net at U1.4 (CANRX): now also U2.2 (CANRX); no longer U2.1 (CANTX)
Changed lines of the file:
@@
 EESchema Schematic File Version 2
+LIBS:can-hat-r1-rescue
 LIBS:power
 LIBS:device
@@
 LIBS:memory
 LIBS:xilinx
-LIBS:special
 LIBS:microcontrollers
 LIBS:dsp
@@
 $EndComp
 $Comp
-L GND #PWR01
+L GND-RESCUE-can-hat-r1 #PWR01
 U 1 1 54F16161
 P 2050 3950
@@
 $EndComp
 $Comp
-L GND #PWR02
+L GND-RESCUE-can-hat-r1 #PWR02
 U 1 1 54F16299
 P 3300 2400
@@
 $EndComp
 $Comp
-L GND #PWR06
+L GND-RESCUE-can-hat-r1 #PWR06
 U 1 1 54F16408
 P 6500 3200
@@
 $EndComp
 $Comp
-L GND #PWR07
+L GND-RESCUE-can-hat-r1 #PWR07
 U 1 1 54F16654
 P 4000 5600
@@
 $EndComp
 $Comp
-L GND #PWR08
+L GND-RESCUE-can-hat-r1 #PWR08
 U 1 1 54F16D07
 P 8650 6600
@@
 ID_SC
 $Comp
-L R R1
+L R-RESCUE-can-hat-r1 R1
 U 1 1 54F17782
 P 7950 1250
@@
 $EndComp
 $Comp
-L R R2
+L R-RESCUE-can-hat-r1 R2
 U 1 1 54F177FE
 P 8250 1250
@@
 $EndComp
 $Comp
-L R R3
+L R-RESCUE-can-hat-r1 R3
 U 1 1 54F1781F
 P 8550 1250
@@
 $EndComp
 $Comp
-L R R4
+L R-RESCUE-can-hat-r1 R4
 U 1 1 54F1783C
 P 8850 1250
@@
 $EndComp
 $Comp
-L R R5
+L R-RESCUE-can-hat-r1 R5
 U 1 1 54F17869
 P 9150 1250
@@
 $EndComp
 $Comp
-L R R6
+L R-RESCUE-can-hat-r1 R6
 U 1 1 54F17882
 P 9450 1250
@@
 $EndComp
 $Comp
-L R R7
+L R-RESCUE-can-hat-r1 R7
 U 1 1 54F1789B
 P 9750 1250
@@
 $EndComp
 $Comp
-L R R8
+L R-RESCUE-can-hat-r1 R8
 U 1 1 54F178B4
 P 10050 1250
@@
 $EndComp
 $Comp
-L R R9
+L R-RESCUE-can-hat-r1 R9
 U 1 1 54F178CD
 P 10350 1250
@@
 $EndComp
 $Comp
-L C C1
+L C-RESCUE-can-hat-r1 C1
 U 1 1 54F184E4
 P 6950 1000
@@
 $EndComp
 $Comp
-L C C2
+L C-RESCUE-can-hat-r1 C2
 U 1 1 54F18509
 P 7250 1000
@@
 $EndComp
 $Comp
-L GND #PWR010
+L GND-RESCUE-can-hat-r1 #PWR010
 U 1 1 54F18522
 P 7100 1400
@@
 $EndComp
 $Comp
-L C C5
+L C-RESCUE-can-hat-r1 C5
 U 1 1 54F18AAE
 P 2350 2550
@@
 $EndComp
 $Comp
-L C C6
+L C-RESCUE-can-hat-r1 C6
 U 1 1 54F18ACD
 P 2650 2550
@@
 $EndComp
 $Comp
-L GND #PWR012
+L GND-RESCUE-can-hat-r1 #PWR012
 U 1 1 54F18B16
 P 2500 2950
@@
 $EndComp
 $Comp
-L R R11
+L R-RESCUE-can-hat-r1 R11
 U 1 1 54F19E16
 P 7600 2700
@@
 $EndComp
 $Comp
-L C C7
+L C-RESCUE-can-hat-r1 C7
 U 1 1 54F19EF2
 P 7950 3000
@@
 $EndComp
 $Comp
-L R R12
+L R-RESCUE-can-hat-r1 R12
 U 1 1 54F19F0F
 P 8400 2700
@@
 $EndComp
 $Comp
-L GND #PWR015
+L GND-RESCUE-can-hat-r1 #PWR015
 U 1 1 54F1A2DC
 P 7950 3300
@@
 $EndComp
 $Comp
-L R R10
+L R-RESCUE-can-hat-r1 R10
 U 1 1 54F1A66B
 P 4150 2150
@@
 $EndComp
 $Comp
-L GND #PWR017
+L GND-RESCUE-can-hat-r1 #PWR017
 U 1 1 54F1A684
 P 4150 2500
@@
 $EndComp
 $Comp
-L C C3
+L C-RESCUE-can-hat-r1 C3
 U 1 1 54F1B073
 P 4400 2400
@@
 $EndComp
 $Comp
-L C C4
+L C-RESCUE-can-hat-r1 C4
 U 1 1 54F1B08C
 P 5200 2400
@@
 $EndComp
 $Comp
-L GND #PWR018
+L GND-RESCUE-can-hat-r1 #PWR018
 U 1 1 54F1B28B
 P 4800 2800
@@
 $EndComp
 $Comp
-L GND #PWR019
+L GND-RESCUE-can-hat-r1 #PWR019
 U 1 1 54F1BC36
 P 1900 7750
@@
 $EndComp
 $Comp
-L C C16
+L C-RESCUE-can-hat-r1 C16
 U 1 1 54F1C097
 P 900 6950
@@
 $EndComp
 $Comp
-L R R19
+L R-RESCUE-can-hat-r1 R19
 U 1 1 54F1C35A
 P 2700 6600
@@
 $EndComp
 $Comp
-L R R20
+L R-RESCUE-can-hat-r1 R20
 U 1 1 54F1C375
 P 3000 6600
@@
 $EndComp
 $Comp
-L R R21
+L R-RESCUE-can-hat-r1 R21
 U 1 1 54F1C394
 P 3300 6600
@@
 Connection ~ 1850 1600
 Connection ~ 1950 1700
-Wire Wire Line
-	5750 1700 4050 1700
-Wire Wire Line
-	5750 1600 4050 1600
 Connection ~ 2050 3850
 Connection ~ 1750 1300
@@
 Connection ~ 2700 6950
 $Comp
-L R R13
+L R-RESCUE-can-hat-r1 R13
 U 1 1 54F1EF87
 P 3300 4900
@@
 $EndComp
 $Comp
-L C C15
+L C-RESCUE-can-hat-r1 C15
 U 1 1 54F1EFA2
 P 2300 5500
@@
 $EndComp
 $Comp
-L R R16
+L R-RESCUE-can-hat-r1 R16
 U 1 1 54F1F062
 P 1750 5500
@@
 $EndComp
 $Comp
-L C C14
+L C-RESCUE-can-hat-r1 C14
 U 1 1 54F1F089
 P 2050 5350
@@
 $EndComp
 $Comp
-L C C8
+L C-RESCUE-can-hat-r1 C8
 U 1 1 54F1F0C2
 P 2050 5100
@@
 	2100 5500 2000 5500
 $Comp
-L GND #PWR022
+L GND-RESCUE-can-hat-r1 #PWR022
 U 1 1 54F1FBA4
 P 1400 5800
@@
 Connection ~ 1400 5500
 $Comp
-L C C9
+L C-RESCUE-can-hat-r1 C9
 U 1 1 54F20342
 P 4300 5100
@@
 Connection ~ 4600 5300
 $Comp
-L R R17
+L R-RESCUE-can-hat-r1 R17
 U 1 1 54F20DC2
 P 1750 5700
@@
 $EndComp
 $Comp
-L R R18
+L R-RESCUE-can-hat-r1 R18
 U 1 1 54F20DE5
 P 2450 5700
@@
 Connection ~ 4000 4900
 $Comp
-L CP C12
+L CP-RESCUE-can-hat-r1 C12
 U 1 1 54F28D96
 P 900 5300
@@
 $EndComp
 $Comp
-L CP C13
+L CP-RESCUE-can-hat-r1 C13
 U 1 1 54F28DAF
 P 1200 5300
@@
 Connection ~ 1200 4800
 $Comp
-L CP C10
+L CP-RESCUE-can-hat-r1 C10
 U 1 1 54F2AC58
 P 5550 5200
@@
 $EndComp
 $Comp
-L CP C11
+L CP-RESCUE-can-hat-r1 C11
 U 1 1 54F2AC77
 P 5800 5200
@@
 Connection ~ 5550 4900
 $Comp
-L GND #PWR025
+L GND-RESCUE-can-hat-r1 #PWR025
 U 1 1 54F2B0C8
 P 5550 5600
@@
 Connection ~ 5550 5500
 $Comp
-L R R22
+L R-RESCUE-can-hat-r1 R22
 U 1 1 54F2B4FD
 P 4700 6600
@@
 $EndComp
 $Comp
-L R R23
+L R-RESCUE-can-hat-r1 R23
 U 1 1 54F2B516
 P 5000 6600
@@
 $EndComp
 $Comp
-L R R24
+L R-RESCUE-can-hat-r1 R24
 U 1 1 54F2B52F
 P 5300 6600
@@
 $EndComp
 $Comp
-L LED D2
+L LED-RESCUE-can-hat-r1 D2
 U 1 1 54F2B548
 P 4700 7250
@@
 $EndComp
 $Comp
-L LED D3
+L LED-RESCUE-can-hat-r1 D3
 U 1 1 54F2B573
 P 5000 7250
@@
 $EndComp
 $Comp
-L LED D4
+L LED-RESCUE-can-hat-r1 D4
 U 1 1 54F2B596
 P 5300 7250
@@
 $EndComp
 $Comp
-L GND #PWR026
+L GND-RESCUE-can-hat-r1 #PWR026
 U 1 1 54F2B5B1
 P 5000 7650
@@
 	7300 4850 7300 5000
 $Comp
-L R R14
+L R-RESCUE-can-hat-r1 R14
 U 1 1 54F2F417
 P 6400 5250
@@
 $EndComp
 $Comp
-L R R15
+L R-RESCUE-can-hat-r1 R15
 U 1 1 54F2F434
 P 7300 5250
@@
 	6400 5500 6400 5700
 $Comp
-L GND #PWR032
+L GND-RESCUE-can-hat-r1 #PWR032
 U 1 1 54F2F837
 P 6400 5700
@@
 	0    -1   -1   0
 $EndComp
+Wire Wire Line
+	4050 1600 4600 1600
+Wire Wire Line
+	4600 1600 4600 1550
+Wire Wire Line
+	4600 1550 4700 1550
+Wire Wire Line
+	4700 1550 4700 1700
+Wire Wire Line
+	4700 1700 5750 1700
+Wire Wire Line
+	5750 1600 4650 1600
+Wire Wire Line
+	4650 1600 4650 1700
+Wire Wire Line
+	4650 1700 4050 1700
 $EndSCHEMATC
